File: PCB/usbcpd.kicad_sch (KiCad schematic)
At the start: 0 parts

Commit message: ok mcu
Parts:
- added U?: STUSB4500QTR, Package_DFN_QFN:QFN-24-1EP_4x4mm_P0.5mm_EP2.7x2.7mm, symbol Interface_USB:STUSB4500QTR
Connections:
- new net: U?.10 (GND), U?.25 (GND)
Changed lines of the file:
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@@
     (effects (font (size 1.27 1.27)) (justify left))
   )
+  (symbol (lib_id "Interface_USB:STUSB4500QTR") (at 152.4 102.87 0) (unit 1)
+    (in_bom yes) (on_board yes) (fields_autoplaced)
+    (property "Reference" "U?" (id 0) (at 154.4194 125.73 0)
+      (effects (font (size 1.27 1.27)) (justify left))
+    )
+    (property "Value" "STUSB4500QTR" (id 1) (at 154.4194 128.27 0)
+      (effects (font (size 1.27 1.27)) (justify left))
+    )
+    (property "Footprint" "Package_DFN_QFN:QFN-24-1EP_4x4mm_P0.5mm_EP2.7x2.7mm" (id 2) (at 152.4 102.87 0)
+      (effects (font (size 1.27 1.27)) hide)
+    )
+    (property "Datasheet" "https://www.st.com/resource/en/datasheet/stusb4500.pdf" (id 3) (at 152.4 102.87 0)
+      (effects (font (size 1.27 1.27)) hide)
+    )
+    (pin "1")
+    (pin "10")
+    (pin "11")
+    (pin "12")
+    (pin "13")
+    (pin "14")
+    (pin "15")
+    (pin "16")
+    (pin "17")
+    (pin "18")
+    (pin "19")
+    (pin "2")
+    (pin "20")
+    (pin "21")
+    (pin "22")
+    (pin "23")
+    (pin "24")
+    (pin "25")
+    (pin "3")
+    (pin "4")
+    (pin "5")
+    (pin "6")
+    (pin "7")
+    (pin "8")
+    (pin "9")
+  )
 )

Commit message: almost ok stusb
Parts:
- added C?: 4.7u, symbol Device:C
- added C? (x4): 1u, symbol Device:C
- added C?: 100n, symbol Device:C
- added D?: ESDA25P35, symbol Device:D_Zener
- added D?: RB501SM-30FHT2R, Diode_SMD:D_SOD-523, symbol Device:D_Schottky
- added J?: USB_C_Receptacle_USB2.0, symbol Connector:USB_C_Receptacle_USB2.0
- added Q?: SSM6J507NU, symbol Device:Q_PMOS_DGS
- added R? (x4): 100k, symbol Device:R
- added R? (x2): 1k, symbol Device:R
- added R?: 18k, symbol Device:R
- added R?: 100, symbol Device:R
- added R?: 470, symbol Device:R
Connections:
- net V_{USB}: now also C?.2, Q?.1 (D), R?.2
- net CC1: now reaches U?.1 (CC1DB)
- net CC1: now also U?.2 (CC1), J?.A5 (CC1)
- net GND: now reaches U?.10 (GND), U?.25 (GND)
- net GND: now also U?.22 (VSYS), C?.1, C?.2, C?.2, C?.2, C?.2, D?.2 (A), J?.A1 (GND), J?.A12 (GND), J?.B1 (GND), J?.B12 (GND), J?.S1 (SHIELD), R?.1, R?.1, R?.1
- net at U?.12 (ADDR0): now also R?.2
- net at U?.13 (ADDR1): now also R?.2
- net at U?.16 (VBUS_EN_SNK): now also R?.1
- net at U?.18 (VBUS_VS_DISCH): now also R?.2
- net at U?.21 (VREG_1V2): now also C?.1
- net at U?.23 (VREG_2V7): now also C?.1
- net VBUS: now reaches U?.24 (VDD)
- net VBUS: now also C?.1, C?.2, D?.1 (K), D?.2 (A), J?.A4 (VBUS), J?.A9 (VBUS), J?.B4 (VBUS), J?.B9 (VBUS), Q?.3 (S), R?.1, R?.2
- net CC2: now reaches U?.4 (CC2)
- net CC2: now also U?.5 (CC2DB), J?.B5 (CC2)
- net Reset: now reaches U?.6 (RESET)
- net Reset: now also R?.2
- net I2C.SCL: now reaches U?.7 (SCL)
- net I2C.SDA: now reaches U?.8 (SDA)
- net at U?.9 (DISCH): now also R?.1
- new net: Q?.2 (G), R?.1, R?.2, R?.2
- new net: C?.1, D?.1 (K), R?.1, R?.2
- new net: C?.1, R?.1
- no-connect marks 0 -> 5

Commit message: upgrade usb protection + kicad 7
Parts:
- added D1: ESDA25W, Package_TO_SOT_SMD:SOT-323_SC-70, symbol Power_Protection:RCLAMP0502B
- added D2: PACDN042Y3R, Package_TO_SOT_SMD:SOT-23-3, symbol Power_Protection:RCLAMP0502B
- added R1, R2: DNP, symbol Device:R
Connections:
- net CC1: now also D1.1 (K1)
- net CC2: now also D1.2 (K2)
- net GND: now also D1.3 (A), D2.3 (A)
- net at R?.2, U?.12 (ADDR0): now also R1.2
- net at R?.2, U?.13 (ADDR1): now also R2.2
- net 2V7: now reaches C?.1, U?.23 (VREG_2V7)
- net 2V7: now also R1.1, R2.1
- net USB2.D+: now reaches J?.A6 (D+)
- net USB2.D+: now also J?.B6 (D+), D2.2 (K2)
- net USB2.D-: now reaches J?.A7 (D-)
- net USB2.D-: now also J?.B7 (D-), D2.1 (K1)
- net Reset: no longer names the net of R?.2, U?.6 (RESET)
- no-connect marks 5 -> 8
Other:
- moved on the sheet: C?, D?, J?, Q?, R?, U?

Commit message: ok dcdc and power switches
Parts:
- renumbered D1 to D?, D2 to D?, R2 to R?, R1 to R?
Connections:
- net VBUS renamed v_{USB}

Commit message: done with sch before ERC and footprints
Parts:
- gave numbers to parts that had none: 24

Commit message: begin BOM
Parts:
- C1: footprint (none) -> Capacitor_SMD:C_0805_2012Metric; MPN (none) -> GRM219R6YA475KA73D; Manufacturer (none) -> Murata
- C2, C3, C4, C5: footprint (none) -> Capacitor_SMD:C_0603_1608Metric; MPN (none) -> CGA3E1X7R1V105K080AC; Manufacturer (none) -> TDK
- C6: footprint (none) -> Capacitor_SMD:C_0603_1608Metric; MPN (none) -> CGA3E2X7R1H104M080AA; Manufacturer (none) -> TDK
- D2: MPN (none) -> ESDA25W; Manufacturer (none) -> STMicroelectronics
- D3: footprint (none) -> Diode_SMD:D_0603_1608Metric; MPN (none) -> ESDA25P35-1U1M; Manufacturer (none) -> STMicroelectronics
- D4: MPN (none) -> PACDN042Y3R; Manufacturer (none) -> Onsemi
- D5: MPN (none) -> RB501SM-30FHT2R; Manufacturer (none) -> ROHM
Changed lines of the file:
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@@
+      (effects (font (size 1.27 1.27)) hide)
+    )
+    (property "MPN" "" (at 210.82 66.04 0)
+      (effects (font (size 1.27 1.27)) hide)
+    )
+    (property "Manufacturer" "" (at 210.82 66.04 0)
       (effects (font (size 1.27 1.27)) hide)
     )
@@
       (effects (font (size 1.27 1.27)) (justify left))
     )
-    (property "Footprint" "" (at 82.2452 85.09 0)
+    (property "Footprint" "Capacitor_SMD:C_0805_2012Metric" (at 82.2452 85.09 0)
       (effects (font (size 1.27 1.27)) hide)
     )
@@
       (effects (font (size 1.27 1.27)) hide)
     )
+    (property "MPN" "GRM219R6YA475KA73D" (at 81.28 81.28 0)
+      (effects (font (size 1.27 1.27)) hide)
+    )
+    (property "Manufacturer" "Murata" (at 81.28 81.28 0)
+      (effects (font (size 1.27 1.27)) hide)
+    )
     (pin "1")
     (pin "2")
@@
       (effects (font (size 1.27 1.27)) (justify left))
     )
-    (property "Footprint" "" (at 144.4752 124.46 0)
+    (property "Footprint" "Capacitor_SMD:C_0603_1608Metric" (at 144.4752 124.46 0)
       (effects (font (size 1.27 1.27)) hide)
     )
@@
       (effects (font (size 1.27 1.27)) hide)
     )
+    (property "MPN" "CGA3E1X7R1V105K080AC" (at 143.51 120.65 0)
+      (effects (font (size 1.27 1.27)) hide)
+    )
+    (property "Manufacturer" "TDK" (at 143.51 120.65 0)
+      (effects (font (size 1.27 1.27)) hide)
+    )
     (pin "1")
     (pin "2")
@@
       (effects (font (size 1.27 1.27)) hide)
     )
+    (property "MPN" "" (at 165.1 137.16 0)
+      (effects (font (size 1.27 1.27)) hide)
+    )
+    (property "Manufacturer" "" (at 165.1 137.16 0)
+      (effects (font (size 1.27 1.27)) hide)
+    )
     (pin "1")
     (pin "2")
@@
       (effects (font (size 1.27 1.27)) (justify left))
     )
-    (property "Footprint" "" (at 242.8748 62.23 0)
+    (property "Footprint" "Capacitor_SMD:C_0603_1608Metric" (at 242.8748 62.23 0)
       (effects (font (size 1.27 1.27)) hide)
     )
@@
       (effects (font (size 1.27 1.27)) hide)
     )
+    (property "MPN" "CGA3E2X7R1H104M080AA " (at 243.84 66.04 0)
+      (effects (font (size 1.27 1.27)) hide)
+    )
+    (property "Manufacturer" "TDK" (at 243.84 66.04 0)
+      (effects (font (size 1.27 1.27)) hide)
+    )
     (pin "1")
     (pin "2")
@@
       (effects (font (size 1.27 1.27)) (justify left))
     )
-    (property "Footprint" "" (at 64.77 81.28 0)
+    (property "Footprint" "Diode_SMD:D_0603_1608Metric" (at 64.77 81.28 0)
       (effects (font (size 1.27 1.27)) hide)
     )
@@
       (effects (font (size 1.27 1.27)) hide)
     )
+    (property "MPN" "ESDA25P35-1U1M" (at 64.77 81.28 0)
+      (effects (font (size 1.27 1.27)) hide)
+    )
+    (property "Manufacturer" "STMicroelectronics " (at 64.77 81.28 0)
+      (effects (font (size 1.27 1.27)) hide)
+    )
     (pin "1")
     (pin "2")
@@
       (effects (font (size 1.27 1.27)) hide)
     )
+    (property "MPN" "" (at 173.99 137.16 0)
+      (effects (font (size 1.27 1.27)) hide)
+    )
+    (property "Manufacturer" "" (at 173.99 137.16 0)
+      (effects (font (size 1.27 1.27)) hide)
+    )
     (pin "1")
     (pin "2")
@@
     )
     (property "Datasheet" "https://www.st.com/resource/en/datasheet/stusb4500.pdf" (at 191.77 113.03 0)
+      (effects (font (size 1.27 1.27)) hide)
+    )
+    (property "MPN" "" (at 191.77 113.03 0)
+      (effects (font (size 1.27 1.27)) hide)
+    )
+    (property "Manufacturer" "" (at 191.77 113.03 0)
       (effects (font (size 1.27 1.27)) hide)
     )
@@
       (effects (font (size 1.27 1.27)) (justify left))
     )
-    (property "Footprint" "" (at 185.42 76.5048 0)
+    (property "Footprint" "Capacitor_SMD:C_0603_1608Metric" (at 185.42 76.5048 0)
       (effects (font (size 1.27 1.27)) hide)
     )
@@
       (effects (font (size 1.27 1.27)) hide)
     )
+    (property "MPN" "CGA3E1X7R1V105K080AC" (at 181.61 77.47 0)
+      (effects (font (size 1.27 1.27)) hide)
+    )
+    (property "Manufacturer" "TDK" (at 181.61 77.47 0)
+      (effects (font (size 1.27 1.27)) hide)
+    )
     (pin "1")
     (pin "2")
@@
     )
     (property "Datasheet" "https://www.usb.org/sites/default/files/documents/usb_type-c.zip" (at 53.34 114.3 0)
+      (effects (font (size 1.27 1.27)) hide)
+    )
+    (property "MPN" "" (at 49.53 114.3 0)
+      (effects (font (size 1.27 1.27)) hide)
+    )
+    (property "Manufacturer" "" (at 49.53 114.3 0)
       (effects (font (size 1.27 1.27)) hide)
     )
@@
       (effects (font (size 1.27 1.27)) hide)
     )
+    (property "MPN" "ESDA25W" (at 57.15 167.64 0)
+      (effects (font (size 1.27 1.27)) hide)
+    )
+    (property "Manufacturer" "STMicroelectronics " (at 57.15 167.64 0)
+      (effects (font (size 1.27 1.27)) hide)
+    )
     (pin "3")
     (pin "1")
@@
       (effects (font (size 1.27 1.27)) hide)
     )
+    (property "MPN" "" (at 170.18 115.57 0)
+      (effects (font (size 1.27 1.27)) hide)
+    )
+    (property "Manufacturer" "" (at 170.18 115.57 0)
+      (effects (font (size 1.27 1.27)) hide)
+    )
     (pin "1")
     (pin "2")
@@
       (effects (font (size 1.27 1.27)) (justify left))
     )
-    (property "Footprint" "" (at 212.09 76.5048 0)
+    (property "Footprint" "Capacitor_SMD:C_0603_1608Metric" (at 212.09 76.5048 0)
       (effects (font (size 1.27 1.27)) hide)
     )
     (property "Datasheet" "~" (at 208.28 77.47 0)
+      (effects (font (size 1.27 1.27)) hide)
+    )
+    (property "MPN" "CGA3E1X7R1V105K080AC" (at 208.28 77.47 0)
+      (effects (font (size 1.27 1.27)) hide)
+    )
+    (property "Manufacturer" "TDK" (at 208.28 77.47 0)
       (effects (font (size 1.27 1.27)) hide)
     )
@@
       (effects (font (size 1.27 1.27)) hide)
     )
+    (property "MPN" "PACDN042Y3R" (at 72.39 127 0)
+      (effects (font (size 1.27 1.27)) hide)
+    )
+    (property "Manufacturer" "Onsemi" (at 72.39 127 0)
+      (effects (font (size 1.27 1.27)) hide)
+    )
     (pin "3")
     (pin "1")
@@
       (effects (font (size 1.27 1.27)) (justify left))
     )
-    (property "Footprint" "" (at 212.09 84.1248 0)
+    (property "Footprint" "Capacitor_SMD:C_0603_1608Metric" (at 212.09 84.1248 0)
       (effects (font (size 1.27 1.27)) hide)
     )
     (property "Datasheet" "~" (at 208.28 85.09 0)
+      (effects (font (size 1.27 1.27)) hide)
+    )
+    (property "MPN" "CGA3E1X7R1V105K080AC" (at 208.28 85.09 0)
+      (effects (font (size 1.27 1.27)) hide)
+    )
+    (property "Manufacturer" "TDK" (at 208.28 85.09 0)
       (effects (font (size 1.27 1.27)) hide)
     )
@@
       (effects (font (size 1.27 1.27)) hide)
     )
+    (property "MPN" "RB501SM-30FHT2R" (at 143.51 110.49 0)
+      (effects (font (size 1.27 1.27)) hide)
+    )
+    (property "Manufacturer" "ROHM" (at 143.51 110.49 0)
+      (effects (font (size 1.27 1.27)) hide)
+    )
     (pin "1")
     (pin "2")
@@
       (effects (font (size 1.27 1.27)) hide)
     )
+    (property "MPN" "" (at 224.79 63.5 0)
+      (effects (font (size 1.27 1.27)) hide)
+    )
+    (property "Manufacturer" "" (at 224.79 63.5 0)
+      (effects (font (size 1.27 1.27)) hide)
+    )
     (pin "1")
     (pin "2")
@@
     )
     (property "Datasheet" "~" (at 224.79 80.01 0)
+      (effects (font (size 1.27 1.27)) hide)
+    )
+    (property "MPN" "" (at 224.79 80.01 0)
+      (effects (font (size 1.27 1.27)) hide)
+    )
+    (property "Manufacturer" "" (at 224.79 80.01 0)
       (effects (font (size 1.27 1.27)) hide)
     )
@@
       (effects (font (size 1.27 1.27)) hide)
     )
+    (property "MPN" "" (at 149.86 137.16 0)
+      (effects (font (size 1.27 1.27)) hide)
+    )
+    (property "Manufacturer" "" (at 149.86 137.16 0)
+      (effects (font (size 1.27 1.27)) hide)
+    )
     (pin "1")
     (pin "2")
@@
     )
     (property "Datasheet" "~" (at 236.22 69.85 0)
+      (effects (font (size 1.27 1.27)) hide)
+    )
+    (property "MPN" "" (at 236.22 69.85 0)
+      (effects (font (size 1.27 1.27)) hide)
+    )
+    (property "Manufacturer" "" (at 236.22 69.85 0)
       (effects (font (size 1.27 1.27)) hide)
     )
@@
       (effects (font (size 1.27 1.27)) hide)
     )
+    (property "MPN" "" (at 142.24 137.16 0)
+      (effects (font (size 1.27 1.27)) hide)
+    )
+    (property "Manufacturer" "" (at 142.24 137.16 0)
+      (effects (font (size 1.27 1.27)) hide)
+    )
     (pin "1")
     (pin "2")
@@
       (effects (font (size 1.27 1.27)) hide)
     )
+    (property "MPN" "" (at 153.67 109.22 0)
+      (effects (font (size 1.27 1.27)) hide)
+    )
+    (property "Manufacturer" "" (at 153.67 109.22 0)
+      (effects (font (size 1.27 1.27)) hide)
+    )
     (pin "1")
     (pin "2")
@@
       (effects (font (size 1.27 1.27)) hide)
     )
+    (property "MPN" "" (at 162.56 100.33 0)
+      (effects (font (size 1.27 1.27)) hide)
+    )
+    (property "Manufacturer" "" (at 162.56 100.33 0)
+      (effects (font (size 1.27 1.27)) hide)
+    )
     (pin "1")
     (pin "2")
@@
       (effects (font (size 1.27 1.27)) hide)
     )
+    (property "MPN" "" (at 252.73 85.09 0)
+      (effects (font (size 1.27 1.27)) hide)
+    )
+    (property "Manufacturer" "" (at 252.73 85.09 0)
+      (effects (font (size 1.27 1.27)) hide)
+    )
