File: PCB/mcu_dcdc.kicad_sch (KiCad schematic)
At the start: 12 parts, among them U1 MP2456

Commit message: done with sch before ERC and footprints
Parts:
- renumbered C1 to C25, C2 to C26, C3 to C27, C5 to C28, C4 to C29, D2 to D8, D1 to D9, L1 to L3, R1 to R29, R3 to R30, R2 to R31, U1 to U5
Changed lines of the file:
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@@
   (symbol (lib_id "TattooSupplyLib:MP2456") (at 142.24 102.87 0) (unit 1)
     (in_bom yes) (on_board yes) (dnp no) (fields_autoplaced)
-    (property "Reference" "U1" (at 142.24 90.17 0)
+    (property "Reference" "U5" (at 142.24 90.17 0)
       (effects (font (size 1.27 1.27)))
     )
@@
       (project "Tattoo_Supply"
         (path "/036b57f3-323c-4da7-bad2-1c27fa1415e1/dbf96053-22e5-4a99-a7e7-291de2fa9a8f"
-          (reference "U1") (unit 1)
+          (reference "U5") (unit 1)
         )
       )
@@
   (symbol (lib_id "Diode:1N4148W") (at 176.53 96.52 0) (unit 1)
     (in_bom yes) (on_board yes) (dnp no) (fields_autoplaced)
-    (property "Reference" "D1" (at 176.53 91.44 0)
+    (property "Reference" "D9" (at 176.53 91.44 0)
       (effects (font (size 1.27 1.27)))
     )
@@
       (project "Tattoo_Supply"
         (path "/036b57f3-323c-4da7-bad2-1c27fa1415e1/dbf96053-22e5-4a99-a7e7-291de2fa9a8f"
-          (reference "D1") (unit 1)
+          (reference "D9") (unit 1)
         )
       )
@@
   (symbol (lib_id "power:GND") (at 190.5 115.57 0) (unit 1)
     (in_bom yes) (on_board yes) (dnp no) (fields_autoplaced)
-    (property "Reference" "#PWR012" (at 190.5 121.92 0)
+    (property "Reference" "#PWR057" (at 190.5 121.92 0)
       (effects (font (size 1.27 1.27)) hide)
     )
@@
       (project "Tattoo_Supply"
         (path "/036b57f3-323c-4da7-bad2-1c27fa1415e1/dbf96053-22e5-4a99-a7e7-291de2fa9a8f"
-          (reference "#PWR012") (unit 1)
+          (reference "#PWR057") (unit 1)
         )
       )
@@
   (symbol (lib_id "Device:C") (at 167.64 139.7 90) (unit 1)
     (in_bom yes) (on_board yes) (dnp no) (fields_autoplaced)
-    (property "Reference" "C5" (at 167.64 133.35 90)
+    (property "Reference" "C28" (at 167.64 133.35 90)
       (effects (font (size 1.27 1.27)))
     )
@@
       (project "Tattoo_Supply"
         (path "/036b57f3-323c-4da7-bad2-1c27fa1415e1/dbf96053-22e5-4a99-a7e7-291de2fa9a8f"
-          (reference "C5") (unit 1)
+          (reference "C28") (unit 1)
         )
       )
@@
   (symbol (lib_id "Device:C") (at 96.52 102.87 0) (unit 1)
     (in_bom yes) (on_board yes) (dnp no) (fields_autoplaced)
-    (property "Reference" "C1" (at 100.33 102.235 0)
+    (property "Reference" "C25" (at 100.33 102.235 0)
       (effects (font (size 1.27 1.27)) (justify left))
     )
@@
       (project "Tattoo_Supply"
         (path "/036b57f3-323c-4da7-bad2-1c27fa1415e1/dbf96053-22e5-4a99-a7e7-291de2fa9a8f"
-          (reference "C1") (unit 1)
+          (reference "C25") (unit 1)
         )
       )
@@
   (symbol (lib_id "Device:L") (at 176.53 102.87 90) (unit 1)
     (in_bom yes) (on_board yes) (dnp no) (fields_autoplaced)
-    (property "Reference" "L1" (at 176.53 99.06 90)
+    (property "Reference" "L3" (at 176.53 99.06 90)
       (effects (font (size 1.27 1.27)))
     )
@@
       (project "Tattoo_Supply"
         (path "/036b57f3-323c-4da7-bad2-1c27fa1415e1/dbf96053-22e5-4a99-a7e7-291de2fa9a8f"
-          (reference "L1") (unit 1)
+          (reference "L3") (unit 1)
         )
       )
@@
   (symbol (lib_id "power:PWR_FLAG") (at 190.5 92.71 0) (unit 1)
     (in_bom yes) (on_board yes) (dnp no) (fields_autoplaced)
-    (property "Reference" "#FLG01" (at 190.5 90.805 0)
+    (property "Reference" "#FLG04" (at 190.5 90.805 0)
       (effects (font (size 1.27 1.27)) hide)
     )
@@
       (project "Tattoo_Supply"
         (path "/036b57f3-323c-4da7-bad2-1c27fa1415e1/dbf96053-22e5-4a99-a7e7-291de2fa9a8f"
-          (reference "#FLG01") (unit 1)
+          (reference "#FLG04") (unit 1)
         )
       )
@@
   (symbol (lib_id "Device:C") (at 190.5 109.22 0) (unit 1)
     (in_bom yes) (on_board yes) (dnp no) (fields_autoplaced)
-    (property "Reference" "C4" (at 194.31 108.585 0)
+    (property "Reference" "C29" (at 194.31 108.585 0)
       (effects (font (size 1.27 1.27)) (justify left))
     )
@@
       (project "Tattoo_Supply"
         (path "/036b57f3-323c-4da7-bad2-1c27fa1415e1/dbf96053-22e5-4a99-a7e7-291de2fa9a8f"
-          (reference "C4") (unit 1)
+          (reference "C29") (unit 1)
         )
       )
@@
   (symbol (lib_id "Device:R") (at 167.64 129.54 90) (unit 1)
     (in_bom yes) (on_board yes) (dnp no) (fields_autoplaced)
-    (property "Reference" "R2" (at 167.64 124.46 90)
+    (property "Reference" "R31" (at 167.64 124.46 90)
       (effects (font (size 1.27 1.27)))
     )
@@
       (project "Tattoo_Supply"
         (path "/036b57f3-323c-4da7-bad2-1c27fa1415e1/dbf96053-22e5-4a99-a7e7-291de2fa9a8f"
-          (reference "R2") (unit 1)
+          (reference "R31") (unit 1)
         )
       )
@@
   (symbol (lib_id "power:GND") (at 157.48 139.7 0) (unit 1)
     (in_bom yes) (on_board yes) (dnp no) (fields_autoplaced)
-    (property "Reference" "#PWR013" (at 157.48 146.05 0)
+    (property "Reference" "#PWR055" (at 157.48 146.05 0)
       (effects (font (size 1.27 1.27)) hide)
     )
@@
       (project "Tattoo_Supply"
         (path "/036b57f3-323c-4da7-bad2-1c27fa1415e1/dbf96053-22e5-4a99-a7e7-291de2fa9a8f"
-          (reference "#PWR013") (unit 1)
+          (reference "#PWR055") (unit 1)
         )
       )
@@
   (symbol (lib_id "power:GND") (at 96.52 109.22 0) (unit 1)
     (in_bom yes) (on_board yes) (dnp no) (fields_autoplaced)
-    (property "Reference" "#PWR08" (at 96.52 115.57 0)
+    (property "Reference" "#PWR052" (at 96.52 115.57 0)
       (effects (font (size 1.27 1.27)) hide)
     )
@@
       (project "Tattoo_Supply"
         (path "/036b57f3-323c-4da7-bad2-1c27fa1415e1/dbf96053-22e5-4a99-a7e7-291de2fa9a8f"
-          (reference "#PWR08") (unit 1)
+          (reference "#PWR052") (unit 1)
         )
       )
@@
   (symbol (lib_id "Device:C") (at 158.75 96.52 90) (unit 1)
     (in_bom yes) (on_board yes) (dnp no) (fields_autoplaced)
-    (property "Reference" "C3" (at 158.75 90.17 90)
+    (property "Reference" "C27" (at 158.75 90.17 90)
       (effects (font (size 1.27 1.27)))
     )
@@
       (project "Tattoo_Supply"
         (path "/036b57f3-323c-4da7-bad2-1c27fa1415e1/dbf96053-22e5-4a99-a7e7-291de2fa9a8f"
-          (reference "C3") (unit 1)
+          (reference "C27") (unit 1)
         )
       )
@@
   (symbol (lib_id "Device:C") (at 107.95 102.87 0) (unit 1)
     (in_bom yes) (on_board yes) (dnp no) (fields_autoplaced)
-    (property "Reference" "C2" (at 111.76 102.235 0)
+    (property "Reference" "C26" (at 111.76 102.235 0)
       (effects (font (size 1.27 1.27)) (justify left))
     )
@@
       (project "Tattoo_Supply"
         (path "/036b57f3-323c-4da7-bad2-1c27fa1415e1/dbf96053-22e5-4a99-a7e7-291de2fa9a8f"
-          (reference "C2") (unit 1)
+          (reference "C26") (unit 1)
         )
       )
@@
   (symbol (lib_id "Device:D_Schottky") (at 167.64 109.22 270) (unit 1)
     (in_bom yes) (on_board yes) (dnp no) (fields_autoplaced)
-    (property "Reference" "D2" (at 170.18 108.2675 90)
+    (property "Reference" "D8" (at 170.18 108.2675 90)
       (effects (font (size 1.27 1.27)) (justify left))
     )
@@
       (project "Tattoo_Supply"
         (path "/036b57f3-323c-4da7-bad2-1c27fa1415e1/dbf96053-22e5-4a99-a7e7-291de2fa9a8f"
-          (reference "D2") (unit 1)
+          (reference "D8") (unit 1)
         )
       )
@@
   (symbol (lib_id "Device:R") (at 119.38 102.87 0) (unit 1)
     (in_bom yes) (on_board yes) (dnp no) (fields_autoplaced)
-    (property "Reference" "R1" (at 121.92 102.235 0)
+    (property "Reference" "R29" (at 121.92 102.235 0)
       (effects (font (size 1.27 1.27)) (justify left))
     )
@@
       (project "Tattoo_Supply"
         (path "/036b57f3-323c-4da7-bad2-1c27fa1415e1/dbf96053-22e5-4a99-a7e7-291de2fa9a8f"
-          (reference "R1") (unit 1)
+          (reference "R29") (unit 1)
         )
       )
@@
   (symbol (lib_id "power:GND") (at 142.24 116.84 0) (unit 1)
     (in_bom yes) (on_board yes) (dnp no) (fields_autoplaced)
-    (property "Reference" "#PWR010" (at 142.24 123.19 0)
+    (property "Reference" "#PWR054" (at 142.24 123.19 0)
       (effects (font (size 1.27 1.27)) hide)
     )
@@
       (project "Tattoo_Supply"
         (path "/036b57f3-323c-4da7-bad2-1c27fa1415e1/dbf96053-22e5-4a99-a7e7-291de2fa9a8f"
-          (reference "#PWR010") (unit 1)
+          (reference "#PWR054") (unit 1)
         )
       )
@@
   (symbol (lib_id "power:GND") (at 107.95 109.22 0) (unit 1)
     (in_bom yes) (on_board yes) (dnp no) (fields_autoplaced)
-    (property "Reference" "#PWR09" (at 107.95 115.57 0)
+    (property "Reference" "#PWR053" (at 107.95 115.57 0)
       (effects (font (size 1.27 1.27)) hide)
     )
@@
       (project "Tattoo_Supply"
         (path "/036b57f3-323c-4da7-bad2-1c27fa1415e1/dbf96053-22e5-4a99-a7e7-291de2fa9a8f"
-          (reference "#PWR09") (unit 1)
+          (reference "#PWR053") (unit 1)
         )
       )
@@
   (symbol (lib_id "Device:R") (at 157.48 134.62 180) (unit 1)
     (in_bom yes) (on_board yes) (dnp no)
-    (property "Reference" "R3" (at 151.13 133.35 0)
+    (property "Reference" "R30" (at 151.13 133.35 0)
       (effects (font (size 1.27 1.27)) (justify right))
     )
@@
       (project "Tattoo_Supply"
         (path "/036b57f3-323c-4da7-bad2-1c27fa1415e1/dbf96053-22e5-4a99-a7e7-291de2fa9a8f"
-          (reference "R3") (unit 1)
+          (reference "R30") (unit 1)
         )
       )
@@
   (symbol (lib_id "power:GND") (at 167.64 115.57 0) (unit 1)
     (in_bom yes) (on_board yes) (dnp no) (fields_autoplaced)
-    (property "Reference" "#PWR011" (at 167.64 121.92 0)
+    (property "Reference" "#PWR056" (at 167.64 121.92 0)
       (effects (font (size 1.27 1.27)) hide)
     )
@@
       (project "Tattoo_Supply"
         (path "/036b57f3-323c-4da7-bad2-1c27fa1415e1/dbf96053-22e5-4a99-a7e7-291de2fa9a8f"
-          (reference "#PWR011") (unit 1)
-        )
-      )
+          (reference "#PWR056") (unit 1)
+        )
+      )

Commit message: begin BOM
Parts:
- C25: footprint (none) -> Capacitor_SMD:C_0805_2012Metric; MPN (none) -> GRM219R6YA475KA73D; Manufacturer (none) -> Murata
- C26, C27: footprint (none) -> Capacitor_SMD:C_0603_1608Metric; MPN (none) -> CGA3E2X7R1H104M080AA; Manufacturer (none) -> TDK
- C28: footprint (none) -> Capacitor_SMD:C_0603_1608Metric; MPN (none) -> C1608C0G1H470J080AA; Manufacturer (none) -> TDK
- C29: footprint (none) -> Capacitor_SMD:C_0805_2012Metric; MPN (none) -> GRM21BC81C226ME44L; Manufacturer (none) -> Murata
- D8: MPN (none) -> PMEG6010ER,115; Manufacturer (none) -> Nexperia
- D9: MPN (none) -> 1N4148W-7-F; Manufacturer (none) -> Diodes Incorporated
- L3: MPN (none) -> NRS5040T100MMGJ; Manufacturer (none) -> Taiyo Yuden
Changed lines of the file:
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@@
+      (effects (font (size 1.27 1.27)) hide)
+    )
+    (property "MPN" "" (at 142.24 102.87 0)
+      (effects (font (size 1.27 1.27)) hide)
+    )
+    (property "Manufacturer" "" (at 142.24 102.87 0)
       (effects (font (size 1.27 1.27)) hide)
     )
@@
       (effects (font (size 1.27 1.27)) hide)
     )
+    (property "MPN" "1N4148W-7-F" (at 176.53 96.52 0)
+      (effects (font (size 1.27 1.27)) hide)
+    )
+    (property "Manufacturer" "Diodes Incorporated " (at 176.53 96.52 0)
+      (effects (font (size 1.27 1.27)) hide)
+    )
     (pin "1")
     (pin "2")
@@
       (effects (font (size 1.27 1.27)))
     )
-    (property "Footprint" "" (at 171.45 138.7348 0)
+    (property "Footprint" "Capacitor_SMD:C_0603_1608Metric" (at 171.45 138.7348 0)
       (effects (font (size 1.27 1.27)) hide)
     )
@@
       (effects (font (size 1.27 1.27)) hide)
     )
+    (property "MPN" "C1608C0G1H470J080AA " (at 167.64 139.7 0)
+      (effects (font (size 1.27 1.27)) hide)
+    )
+    (property "Manufacturer" "TDK" (at 167.64 139.7 0)
+      (effects (font (size 1.27 1.27)) hide)
+    )
     (pin "1")
     (pin "2")
@@
       (effects (font (size 1.27 1.27)) (justify left))
     )
-    (property "Footprint" "" (at 97.4852 106.68 0)
+    (property "Footprint" "Capacitor_SMD:C_0805_2012Metric" (at 97.4852 106.68 0)
       (effects (font (size 1.27 1.27)) hide)
     )
@@
       (effects (font (size 1.27 1.27)) hide)
     )
+    (property "MPN" "GRM219R6YA475KA73D" (at 96.52 102.87 0)
+      (effects (font (size 1.27 1.27)) hide)
+    )
+    (property "Manufacturer" "Murata" (at 96.52 102.87 0)
+      (effects (font (size 1.27 1.27)) hide)
+    )
     (pin "1")
     (pin "2")
@@
       (effects (font (size 1.27 1.27)) hide)
     )
+    (property "MPN" "NRS5040T100MMGJ" (at 176.53 102.87 0)
+      (effects (font (size 1.27 1.27)) hide)
+    )
+    (property "Manufacturer" "Taiyo Yuden" (at 176.53 102.87 0)
+      (effects (font (size 1.27 1.27)) hide)
+    )
     (pin "1")
     (pin "2")
@@
       (effects (font (size 1.27 1.27)) (justify left))
     )
-    (property "Footprint" "" (at 191.4652 113.03 0)
+    (property "Footprint" "Capacitor_SMD:C_0805_2012Metric" (at 191.4652 113.03 0)
       (effects (font (size 1.27 1.27)) hide)
     )
@@
       (effects (font (size 1.27 1.27)) hide)
     )
+    (property "MPN" "GRM21BC81C226ME44L" (at 190.5 109.22 0)
+      (effects (font (size 1.27 1.27)) hide)
+    )
+    (property "Manufacturer" "Murata" (at 190.5 109.22 0)
+      (effects (font (size 1.27 1.27)) hide)
+    )
     (pin "1")
     (pin "2")
@@
       (effects (font (size 1.27 1.27)) hide)
     )
+    (property "MPN" "" (at 167.64 129.54 0)
+      (effects (font (size 1.27 1.27)) hide)
+    )
+    (property "Manufacturer" "" (at 167.64 129.54 0)
+      (effects (font (size 1.27 1.27)) hide)
+    )
     (pin "1")
     (pin "2")
@@
       (effects (font (size 1.27 1.27)))
     )
-    (property "Footprint" "" (at 162.56 95.5548 0)
+    (property "Footprint" "Capacitor_SMD:C_0603_1608Metric" (at 162.56 95.5548 0)
       (effects (font (size 1.27 1.27)) hide)
     )
@@
       (effects (font (size 1.27 1.27)) hide)
     )
+    (property "MPN" "CGA3E2X7R1H104M080AA " (at 158.75 96.52 0)
+      (effects (font (size 1.27 1.27)) hide)
+    )
+    (property "Manufacturer" "TDK" (at 158.75 96.52 0)
+      (effects (font (size 1.27 1.27)) hide)
+    )
     (pin "1")
     (pin "2")
@@
       (effects (font (size 1.27 1.27)) (justify left))
     )
-    (property "Footprint" "" (at 108.9152 106.68 0)
+    (property "Footprint" "Capacitor_SMD:C_0603_1608Metric" (at 108.9152 106.68 0)
       (effects (font (size 1.27 1.27)) hide)
     )
@@
       (effects (font (size 1.27 1.27)) hide)
     )
+    (property "MPN" "CGA3E2X7R1H104M080AA " (at 107.95 102.87 0)
+      (effects (font (size 1.27 1.27)) hide)
+    )
+    (property "Manufacturer" "TDK" (at 107.95 102.87 0)
+      (effects (font (size 1.27 1.27)) hide)
+    )
     (pin "1")
     (pin "2")
@@
       (effects (font (size 1.27 1.27)) hide)
     )
+    (property "MPN" "PMEG6010ER,115" (at 167.64 109.22 0)
+      (effects (font (size 1.27 1.27)) hide)
+    )
+    (property "Manufacturer" "Nexperia" (at 167.64 109.22 0)
+      (effects (font (size 1.27 1.27)) hide)
+    )
     (pin "1")
     (pin "2")
@@
     )
     (property "Datasheet" "~" (at 119.38 102.87 0)
+      (effects (font (size 1.27 1.27)) hide)
+    )
+    (property "MPN" "" (at 119.38 102.87 0)
+      (effects (font (size 1.27 1.27)) hide)
+    )
+    (property "Manufacturer" "" (at 119.38 102.87 0)
       (effects (font (size 1.27 1.27)) hide)
     )
@@
       (effects (font (size 1.27 1.27)) hide)
     )
+    (property "MPN" "" (at 157.48 134.62 0)
+      (effects (font (size 1.27 1.27)) hide)
+    )
+    (property "Manufacturer" "" (at 157.48 134.62 0)
+      (effects (font (size 1.27 1.27)) hide)
+    )

Commit message: Resistors ok in BOM
Parts:
- R29: value 500k -> 499k; footprint (none) -> Resistor_SMD:R_0603_1608Metric; MPN (none) -> ERJ-3EKF4993V; Manufacturer (none) -> Panasonic
- R30: footprint (none) -> Resistor_SMD:R_0603_1608Metric; MPN (none) -> ERJ-3EKF4022V; Manufacturer (none) -> Panasonic
- R31: footprint (none) -> Resistor_SMD:R_0603_1608Metric; MPN (none) -> ERJ-3EKF1243V; Manufacturer (none) -> Panasonic
Changed lines of the file:
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@@
       (effects (font (size 1.27 1.27)))
     )
-    (property "Footprint" "" (at 167.64 131.318 90)
+    (property "Footprint" "Resistor_SMD:R_0603_1608Metric" (at 167.64 131.318 90)
       (effects (font (size 1.27 1.27)) hide)
     )
@@
       (effects (font (size 1.27 1.27)) hide)
     )
-    (property "MPN" "" (at 167.64 129.54 0)
-      (effects (font (size 1.27 1.27)) hide)
-    )
-    (property "Manufacturer" "" (at 167.64 129.54 0)
+    (property "MPN" "ERJ-3EKF1243V" (at 167.64 129.54 0)
+      (effects (font (size 1.27 1.27)) hide)
+    )
+    (property "Manufacturer" "Panasonic" (at 167.64 129.54 0)
       (effects (font (size 1.27 1.27)) hide)
     )
@@
       (effects (font (size 1.27 1.27)) (justify left))
     )
-    (property "Value" "500k" (at 121.92 104.775 0)
-      (effects (font (size 1.27 1.27)) (justify left))
-    )
-    (property "Footprint" "" (at 117.602 102.87 90)
+    (property "Value" "499k" (at 121.92 104.775 0)
+      (effects (font (size 1.27 1.27)) (justify left))
+    )
+    (property "Footprint" "Resistor_SMD:R_0603_1608Metric" (at 117.602 102.87 90)
       (effects (font (size 1.27 1.27)) hide)
     )
@@
       (effects (font (size 1.27 1.27)) hide)
     )
-    (property "MPN" "" (at 119.38 102.87 0)
-      (effects (font (size 1.27 1.27)) hide)
-    )
-    (property "Manufacturer" "" (at 119.38 102.87 0)
+    (property "MPN" "ERJ-3EKF4993V" (at 119.38 102.87 0)
+      (effects (font (size 1.27 1.27)) hide)
+    )
+    (property "Manufacturer" "Panasonic" (at 119.38 102.87 0)
       (effects (font (size 1.27 1.27)) hide)
     )
@@
       (effects (font (size 1.27 1.27)) (justify right))
     )
-    (property "Footprint" "" (at 159.258 134.62 90)
+    (property "Footprint" "Resistor_SMD:R_0603_1608Metric" (at 159.258 134.62 90)
       (effects (font (size 1.27 1.27)) hide)
     )
@@
       (effects (font (size 1.27 1.27)) hide)
     )
-    (property "MPN" "" (at 157.48 134.62 0)
-      (effects (font (size 1.27 1.27)) hide)
-    )
-    (property "Manufacturer" "" (at 157.48 134.62 0)
-      (effects (font (size 1.27 1.27)) hide)
-    )
+    (property "MPN" " ERJ-3EKF4022V" (at 157.48 134.62 0)
+      (effects (font (size 1.27 1.27)) hide)
+    )
+    (property "Manufacturer" "Panasonic" (at 157.48 134.62 0)
+      (effects (font (size 1.27 1.27)) hide)
+    )

Commit message: bom almost finished
Parts:
- U5: MPN (none) -> MP2456GJ-Z; Manufacturer (none) -> Monolithic Power Systems
Changed lines of the file:
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@@
       (effects (font (size 1.27 1.27)) hide)
     )
-    (property "MPN" "" (at 142.24 102.87 0)
+    (property "MPN" "MP2456GJ-Z" (at 142.24 102.87 0)
       (effects (font (size 1.27 1.27)) hide)
     )
-    (property "Manufacturer" "" (at 142.24 102.87 0)
+    (property "Manufacturer" "Monolithic Power Systems" (at 142.24 102.87 0)
       (effects (font (size 1.27 1.27)) hide)
     )
@@
       (effects (font (size 1.27 1.27)) hide)
     )
-    (property "Sim.Device" "D" (at 176.53 96.52 0)
-      (effects (font (size 1.27 1.27)) hide)
-    )
-    (property "Sim.Pins" "1=K 2=A" (at 176.53 96.52 0)
-      (effects (font (size 1.27 1.27)) hide)
-    )

Commit message: update dcdc 3V3 & begin routing
Connections:
- net at C27.1, U5.1 (BST): now also D9.1 (K)
- net at C27.2, D8.1 (K), L3.1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: no longer D9.1 (K)
Changed lines of the file:
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@@
   (junction (at 182.88 102.87) (diameter 0) (color 0 0 0 0)
-  )
-  (junction (at 167.64 96.52) (diameter 0) (color 0 0 0 0)
   )
   (junction (at 182.88 96.52) (diameter 0) (color 0 0 0 0)
@@
   )
   (junction (at 96.52 96.52) (diameter 0) (color 0 0 0 0)
+  )
+  (junction (at 153.67 96.52) (diameter 0) (color 0 0 0 0)
+  )
+  (wire (pts (xy 153.67 87.63) (xy 153.67 96.52))
+    (stroke (width 0) (type default))
   )
   (wire (pts (xy 161.29 129.54) (xy 157.48 129.54))
@@
     (stroke (width 0) (type default))
   )
+  (wire (pts (xy 153.67 96.52) (xy 154.94 96.52))
+    (stroke (width 0) (type default))
+  )
   (wire (pts (xy 163.83 129.54) (xy 161.29 129.54))
     (stroke (width 0) (type default))
@@
     (stroke (width 0) (type default))
   )
+  (wire (pts (xy 170.18 87.63) (xy 153.67 87.63))
+    (stroke (width 0) (type default))
+  )
   (wire (pts (xy 167.64 96.52) (xy 167.64 102.87))
     (stroke (width 0) (type default))
   )
   (wire (pts (xy 96.52 96.52) (xy 96.52 99.06))
-    (stroke (width 0) (type default))
-  )
-  (wire (pts (xy 167.64 96.52) (xy 172.72 96.52))
     (stroke (width 0) (type default))
   )
@@
     (stroke (width 0) (type default))
   )
+  (wire (pts (xy 172.72 96.52) (xy 170.18 96.52))
+    (stroke (width 0) (type default))
+  )
   (wire (pts (xy 157.48 129.54) (xy 157.48 130.81))
     (stroke (width 0) (type default))
@@
     (stroke (width 0) (type default))
   )
-  (wire (pts (xy 152.4 96.52) (xy 154.94 96.52))
+  (wire (pts (xy 152.4 96.52) (xy 153.67 96.52))
     (stroke (width 0) (type default))
   )
@@
     (stroke (width 0) (type default))
   )
+  (wire (pts (xy 170.18 96.52) (xy 170.18 87.63))
+    (stroke (width 0) (type default))
+  )
