File: PCB/dac.kicad_sch (KiCad schematic)
At the start: 8 parts, among them U7 DACx3202

Commit message: ok for dcdc and cleanup
Connections:
- net V_{CC} renamed 3V3
Changed lines of the file:
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@@
 		)
 	)
-	(hierarchical_label "V_{CC}"
+	(hierarchical_label "3V3"
 		(shape input)
 		(at 149.86 73.66 90)
