File: PCB/eeprom.kicad_sch (KiCad schematic)
At the start: 2 parts, among them U11 AT24C02D-STUM-T

Commit message: ok
Changed lines of the file:
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@@
-		)
-	)
-	(hierarchical_label "3V3"
-		(shape input)
-		(at 107.95 58.42 180)
-		(fields_autoplaced yes)
-		(effects
-			(font
-				(size 1.27 1.27)
-			)
-			(justify right)
 		)
 	)
