File: PCB/smps.kicad_sch (KiCad schematic)
At the start: 10 parts, among them U4 LM2576S-ADJ

Commit message: schematic done and bom ok
Parts:
- L2: footprint (none) -> TattooSupplyFootprints:MSS1583
Changed lines of the file:
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@@
+    (stroke (width 0) (type default))
+  )
+  (wire (pts (xy 220.98 85.09) (xy 220.98 88.9))
     (stroke (width 0) (type default))
   )
@@
       (effects (font (size 1.27 1.27)))
     )
-    (property "Footprint" "" (at 146.05 88.9 0)
+    (property "Footprint" "TattooSupplyFootprints:MSS1583" (at 146.05 88.9 0)
       (effects (font (size 1.27 1.27)) hide)
     )
@@
         )
       )
+    )
+  )
+  (symbol (lib_id "power:PWR_FLAG") (at 220.98 85.09 0) (unit 1)
+    (in_bom yes) (on_board yes) (dnp no) (fields_autoplaced)
+    (property "Reference" "#FLG08" (at 220.98 83.185 0)
+      (effects (font (size 1.27 1.27)) hide)
+    )
+    (property "Value" "PWR_FLAG" (at 220.98 81.28 0)
+      (effects (font (size 1.27 1.27)))
+    )
+    (property "Footprint" "" (at 220.98 85.09 0)
+      (effects (font (size 1.27 1.27)) hide)
+    )
+    (property "Datasheet" "~" (at 220.98 85.09 0)
+      (effects (font (size 1.27 1.27)) hide)
+    )
+    (pin "1")
+    (instances
+      (project "Tattoo_Supply"
+        (path "/036b57f3-323c-4da7-bad2-1c27fa1415e1/ceea0ffd-34e8-4863-a5ab-807ee81bbc9d"
+          (reference "#FLG08") (unit 1)
+        )
+        (path "/036b57f3-323c-4da7-bad2-1c27fa1415e1/0bfe1b8d-2b80-49bc-95c3-66c860b9d04a"
+          (reference "#FLG07") (unit 1)
+        )
+      )

Commit message: ok better cap
Parts:
- C22, C23: footprint TattooSupplyFootprints:CPL_12.5_14 -> Capacitor_SMD:CP_Elec_8x10; MPN 865060562009 -> EMZS350ARA471MHA0G; Manufacturer Wurth Elektronik -> United Chemi-Con
Changed lines of the file:
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@@
       (effects (font (size 1.27 1.27)) (justify left))
     )
-    (property "Footprint" "TattooSupplyFootprints:CPL_12.5_14" (at 176.2252 102.87 0)
+    (property "Footprint" "Capacitor_SMD:CP_Elec_8x10" (at 176.2252 102.87 0)
       (effects (font (size 1.27 1.27)) hide)
     )
@@
       (effects (font (size 1.27 1.27)) hide)
     )
-    (property "MPN" "865060562009" (at 175.26 99.06 0)
-      (effects (font (size 1.27 1.27)) hide)
-    )
-    (property "Manufacturer" "Wurth Elektronik" (at 175.26 99.06 0)
+    (property "MPN" "EMZS350ARA471MHA0G" (at 175.26 99.06 0)
+      (effects (font (size 1.27 1.27)) hide)
+    )
+    (property "Manufacturer" "United Chemi-Con " (at 175.26 99.06 0)
       (effects (font (size 1.27 1.27)) hide)
     )
@@
       (effects (font (size 1.27 1.27)) (justify left))
     )
-    (property "Footprint" "TattooSupplyFootprints:CPL_12.5_14" (at 159.7152 102.87 0)
+    (property "Footprint" "Capacitor_SMD:CP_Elec_8x10" (at 159.7152 102.87 0)
       (effects (font (size 1.27 1.27)) hide)
     )
@@
       (effects (font (size 1.27 1.27)) hide)
     )
-    (property "MPN" "865060562009" (at 158.75 99.06 0)
-      (effects (font (size 1.27 1.27)) hide)
-    )
-    (property "Manufacturer" "Wurth Elektronik" (at 158.75 99.06 0)
-      (effects (font (size 1.27 1.27)) hide)
-    )
+    (property "MPN" "EMZS350ARA471MHA0G" (at 158.75 99.06 0)
+      (effects (font (size 1.27 1.27)) hide)
+    )
+    (property "Manufacturer" "United Chemi-Con " (at 158.75 99.06 0)
+      (effects (font (size 1.27 1.27)) hide)
+    )

Commit message: change by rp2040
Parts:
- renumbered C24 to C10, C21 to C7, C22 to C8, C23 to C9, D7 to D6, L2 to L1, R26 to R13, R27 to R14, R28 to R15, U4 to U2
Changed lines of the file:
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@@
 		(dnp no)
 		(fields_autoplaced yes)
-		(property "Reference" "R26"
+		(property "Reference" "R13"
 			(at 223.52 92.7099 0)
 			(effects
@@
 		(dnp no)
 		(fields_autoplaced yes)
-		(property "Reference" "#PWR047"
+		(property "Reference" "#PWR028"
 			(at 134.62 111.76 0)
 			(effects
@@
 		(on_board yes)
 		(dnp no)
-		(property "Reference" "R28"
+		(property "Reference" "R15"
 			(at 231.14 104.14 90)
 			(effects
@@
 		(dnp no)
 		(fields_autoplaced yes)
-		(property "Reference" "U4"
+		(property "Reference" "U2"
 			(at 115.57 76.2 0)
 			(effects
@@
 		(dnp no)
 		(fields_autoplaced yes)
-		(property "Reference" "#PWR050"
+		(property "Reference" "#PWR031"
 			(at 191.77 111.76 0)
 			(effects
@@
 		(dnp no)
 		(fields_autoplaced yes)
-		(property "Reference" "D7"
+		(property "Reference" "D6"
 			(at 137.16 97.4724 90)
 			(effects
@@
 		(dnp no)
 		(fields_autoplaced yes)
-		(property "Reference" "C23"
+		(property "Reference" "C9"
 			(at 179.07 96.9009 0)
 			(effects
@@
 		(dnp no)
 		(fields_autoplaced yes)
-		(property "Reference" "C21"
+		(property "Reference" "C7"
 			(at 72.39 96.9009 0)
 			(effects
@@
 		(dnp no)
 		(fields_autoplaced yes)
-		(property "Reference" "R27"
+		(property "Reference" "R14"
 			(at 223.52 105.4099 0)
 			(effects
@@
 		(dnp no)
 		(fields_autoplaced yes)
-		(property "Reference" "#PWR045"
+		(property "Reference" "#PWR026"
 			(at 68.58 111.76 0)
 			(effects
@@
 		(dnp no)
 		(fields_autoplaced yes)
-		(property "Reference" "#PWR048"
+		(property "Reference" "#PWR029"
 			(at 158.75 111.76 0)
 			(effects
@@
 		(dnp no)
 		(fields_autoplaced yes)
-		(property "Reference" "#PWR049"
+		(property "Reference" "#PWR030"
 			(at 175.26 111.76 0)
 			(effects
@@
 		(dnp no)
 		(fields_autoplaced yes)
-		(property "Reference" "L2"
+		(property "Reference" "L1"
 			(at 146.05 82.55 90)
 			(effects
@@
 		(dnp no)
 		(fields_autoplaced yes)
-		(property "Reference" "#PWR046"
+		(property "Reference" "#PWR027"
 			(at 115.57 111.76 0)
 			(effects
@@
 		(dnp no)
 		(fields_autoplaced yes)
-		(property "Reference" "#PWR051"
+		(property "Reference" "#PWR032"
 			(at 220.98 119.38 0)
 			(effects
@@
 		(dnp no)
 		(fields_autoplaced yes)
-		(property "Reference" "C22"
+		(property "Reference" "C8"
 			(at 162.56 96.9009 0)
 			(effects
@@
 		(dnp no)
 		(fields_autoplaced yes)
-		(property "Reference" "#FLG08"
+		(property "Reference" "#FLG07"
 			(at 220.98 83.185 0)
 			(effects
@@
 		(dnp no)
 		(fields_autoplaced yes)
-		(property "Reference" "C24"
+		(property "Reference" "C10"
 			(at 195.58 97.7899 0)
 			(effects

Commit message: ok for dcdc and cleanup
Parts:
- removed C10: 1u, Capacitor_SMD:C_0603_1608Metric, symbol Device:C
- removed C7: 100u/35V, Capacitor_SMD:CP_Elec_6.3x7.7, symbol Device:C_Polarized
- removed C8, C9: 470u/35V, Capacitor_SMD:CP_Elec_8x10, symbol Device:C_Polarized
- removed D6: PMEG4050EP,115, Diode_SMD:D_SOD-128, symbol Device:D_Schottky
- removed L1: MSS1583-154KED, TattooSupplyFootprints:MSS1583, symbol Device:L
- removed R13: 8.45k, Resistor_SMD:R_0603_1608Metric, symbol Device:R
- removed U2: LM2576S-ADJ, Package_TO_SOT_SMD:TO-263-5_TabPin3, symbol Regulator_Switching:LM2576S-ADJ
- added C22, C23, C42: 22u, symbol Device:C
- added C44: 82p, symbol Device:C
- added C8: 22n, symbol Device:C
- added C9: 100n, symbol Device:C
- added L2: 100u, symbol Device:L
- added R26: 10k, symbol Device:R
- added R28: 127k, symbol Device:R
- added U4: MP2338GTL, Package_TO_SOT_SMD:SOT-583-8, symbol TattooSupplyLib:MP2338GTL
- R14: value 1k -> 562k; footprint Resistor_SMD:R_0603_1608Metric -> (none); MPN ERJ-3EKF1001V -> (none); Manufacturer Panasonic -> (none)
- R15: value 1.65k -> 21.5k; footprint Resistor_SMD:R_0603_1608Metric -> (none); MPN ERJ-3EKF1651V -> (none); Manufacturer Panasonic -> (none)
Connections:
- net GND: now also R15.2, C22.2, C23.2, C42.2, C8.2, U4.4 (GND); no longer R14.2
- net V_{Feedback}: now also R28.2; no longer R15.2
- net V_{IN}: now also C42.1, U4.2 (V_{IN})
- net V_{OUT}: now also R14.1, C22.1, C23.1, C44.1, L2.2
- net at R15.1: now also R14.2, C44.2, R26.2, R28.1; no longer R14.1
- new net: C8.1, U4.7 (SS)
- new net: C9.2, L2.1, U4.3 (SW)
- new net: C9.1, U4.5 (BST)
- new net: R26.1, U4.8 (FB)
- new net ON/~{OFF}: U4.6 (EN)
- no-connect marks 0 -> 1
Other:
- note added: "I_{SAT}=3A"

Commit message: ok
Parts:
- renumbered C22 to C21, C8 to C7, L2 to L1, R14 to R13, U4 to U2
Changed lines of the file:
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@@
 		(dnp no)
 		(fields_autoplaced yes)
-		(property "Reference" "C8"
+		(property "Reference" "C7"
 			(at 130.81 107.9499 0)
 			(effects
@@
 		(dnp no)
 		(fields_autoplaced yes)
-		(property "Reference" "U4"
+		(property "Reference" "U2"
 			(at 149.86 81.28 0)
 			(effects
@@
 		(on_board yes)
 		(dnp no)
-		(property "Reference" "R14"
+		(property "Reference" "R13"
 			(at 200.406 94.488 0)
 			(effects
@@
 		(dnp no)
 		(fields_autoplaced yes)
-		(property "Reference" "L2"
+		(property "Reference" "L1"
 			(at 186.69 83.82 90)
 			(effects
@@
 		(dnp no)
 		(fields_autoplaced yes)
-		(property "Reference" "C22"
+		(property "Reference" "C21"
 			(at 236.22 100.3299 0)
 			(effects
