File: PCB/mcu.kicad_sch (KiCad schematic)
At the start: 29 parts, among them J5 Conn_ST_STDC14, J6 Debug_JTAG, J7 Debug_UART, SW1 Reset, U3 STM32F103C8Tx, Y1 ABM3B-8.000MHZ-B2-T

Commit message: change by rp2040
Parts:
- removed FB1: 600/100MHz, Resistor_SMD:R_0603_1608Metric, symbol Device:FerriteBead
- removed J5: Conn_ST_STDC14, Connector_PinHeader_1.27mm:PinHeader_2x07_P1.27mm_Vertical_SMD, symbol Connector:Conn_ST_STDC14
- removed J7: Debug_UART, Connector_PinHeader_2.54mm:PinHeader_1x03_P2.54mm_Vertical, symbol Connector_Generic:Conn_01x03
- removed JP1: Jumper_3_Open, Connector_PinHeader_2.54mm:PinHeader_1x03_P2.54mm_Vertical, symbol Jumper:Jumper_3_Open
- removed NT1: NetTie_2, NetTie:NetTie-2_SMD_Pad0.5mm, symbol Device:NetTie_2
- removed U3: STM32F103C8Tx, Package_QFP:LQFP-48_7x7mm_P0.5mm, symbol MCU_ST_STM32F1:STM32F103C8Tx
- added SW4: Reset, Button_Switch_SMD:SW_SPST_EVQP2, symbol Switch:SW_Push
- added U10: W25Q16JVZP, Package_SON:WSON-8-1EP_6x5mm_P1.27mm_EP3.4x4.3mm, symbol Memory_Flash:W25Q32JVZP
- added U3: RP2040, Package_DFN_QFN:QFN-56-1EP_7x7mm_P0.4mm_EP3.2x3.2mm, symbol MCU_RaspberryPi:RP2040
- C12, C16: value 20p -> 15p; MPN C0603C200J5HACTU -> (none); Manufacturer Kemet -> (none)
- C15: value 1u -> 100n; MPN CGA3E1X7R1V105K080AC -> CGA3E2X7R1H104M080AA
- C18: value 10n -> 2.2u; MPN GCM188R71H103KA37J -> (none); Manufacturer Murata -> (none)
- R16: value 953 -> 1k; MPN ERJ-3EKF9530V -> (none); Manufacturer Panasonic -> (none)
- R18: value 100k -> 1k; MPN ERJ-3EKF1003V -> (none); Manufacturer Panasonic -> (none); now fitted
- R19: value 100k -> 10k; MPN ERJ-3EKF1003V -> ERJ-3EKF1002V
- R22, R25: value 100k -> 27.4; MPN ERJ-3EKF1003V -> (none); Manufacturer Panasonic -> (none)
- Y1: value ABM3B-8.000MHZ-B2-T -> 12MHz/30ppm; footprint Crystal:Crystal_SMD_Abracon_ABM3B-4Pin_5.0x3.2mm -> Crystal:Crystal_SMD_Abracon_ABM8G-4Pin_3.2x2.5mm; MPN ABM3B-8.000MHZ-B2-T -> ABM8-272-T3
Connections:
- net GNDA is gone; now on net GND: C15.2, C18.2
- net GND: now also SW4.2, U10.4 (GND); no longer R19.2, R22.1
- net SWCLK: now also U3.24 (SWCLK)
- net SWDIO: now also U3.25 (SWD)
- net V_{IN}: no longer C11.1, C14.1, C17.1, C19.1, C20.1, R18.1
- net at R19.1: no longer R18.2
- net USB_DFU: no longer names the net of R25.1
- net USB_DFU: now also U3.46 (USB_DM)
- net VDDA renamed V_{MCU}
- net V_{MCU}: now also C11.1, C14.1, C17.1, C19.1, C20.1, U10.8 (VCC), U3.1 (IOVDD), U3.10 (IOVDD), U3.22 (IOVDD), U3.33 (IOVDD), U3.42 (IOVDD), U3.43 (ADC_AVDD), U3.44 (VREG_IN), U3.48 (USB_VDD), U3.49 (IOVDD)
- new net: R18.1, SW4.1
- new net: R22.1, U3.47 (USB_DP)
- new net 1V1: U3.23 (DVDD), U3.45 (VREG_VOUT), U3.50 (DVDD)
- new net FLASH.CLK: U10.6 (CLK), U3.52 (QSPI_SCLK)
- new net FLASH.IO0: U10.5 (DI(IO0)), U3.53 (QSPI_SD0)
- new net FLASH.IO1: U10.2 (DO(IO1)), U3.55 (QSPI_SD1)
- new net FLASH.IO2: U10.3 (IO2), U3.54 (QSPI_SD2)
- new net FLASH.IO3: U10.7 (IO3), U3.51 (QSPI_SD3)
- new net FLASH.~{CS}: R18.2, U10.1 (~{CS}), U3.56 (QSPI_SS)
- no-connect marks 11 -> 1
Other:
- moved on the sheet: R17, R20, R21, R23, R24

Commit message: ok for rp2040
Parts:
- removed C13, C15: 100n, Capacitor_SMD:C_0603_1608Metric, symbol Device:C
- removed C18: 2.2u, Capacitor_SMD:C_0603_1608Metric, symbol Device:C
- removed J6: Debug_JTAG, Connector_PinHeader_2.54mm:PinHeader_1x04_P2.54mm_Vertical, symbol Connector_Generic:Conn_01x04
- removed R18: 1k, Resistor_SMD:R_0603_1608Metric, symbol Device:R
- removed R19: 10k, Resistor_SMD:R_0603_1608Metric, symbol Device:R
- removed SW1, SW4: Reset, Button_Switch_SMD:SW_SPST_EVQP2, symbol Switch:SW_Push
- removed U10: W25Q16JVZP, Package_SON:WSON-8-1EP_6x5mm_P1.27mm_EP3.4x4.3mm, symbol Memory_Flash:W25Q32JVZP
- added C35, C36, C38, C39: 100n, Capacitor_SMD:C_0603_1608Metric, symbol Device:C
- added C40, C41: 1u, Capacitor_SMD:C_0603_1608Metric, symbol Device:C
- C11: value 4.7u -> 100n; footprint Capacitor_SMD:C_0805_2012Metric -> Capacitor_SMD:C_0603_1608Metric; MPN GRM219R6YA475KA73D -> CGA3E2X7R1H104M080AA; Manufacturer Murata -> TDK
Connections:
- net 1V1: now also C14.1, C17.1, C41.1
- net Analog1: now also U3.38 (GPIO26_ADC0)
- net Analog2: now also U3.39 (GPIO27_ADC1)
- net EN_{SMPS}: now also U3.14 (GPIO11)
- net Footswitch: now also U3.13 (GPIO10)
- net GND: now also U3.57 (GND), C35.2, C36.2, C38.2, C39.2, C40.2, C41.2
- net I2C.SCL: now also U3.3 (GPIO1)
- net I2C.SDA: now also U3.2 (GPIO0)
- net OLED_{DC}: now also U3.8 (GPIO6)
- net OLED_{RES}: now also U3.9 (GPIO7)
- net OSC_{IN}: now also U3.20 (XIN)
- net OSC_{OUT}: now also U3.21 (XOUT)
- net USB.D-: now reaches R25.2
- net USB.D+: now reaches R22.2
- net at U3.11 (GPIO8): now also R23.1
- net at U3.12 (GPIO9): now also R24.1
- net Display.SCK: now reaches U3.4 (GPIO2)
- net Display.MOSI: now reaches U3.5 (GPIO3)
- net Display.MISO: now reaches U3.6 (GPIO4)
- net Display.~{CS}: now reaches U3.7 (GPIO5)
- net SWCLK renamed SWD.SWCLK
- net SWDIO renamed SWD.SWDIO
- net V_{IN} renamed 3V3
- net 3V3: now also C11.1, C19.1, C20.1, U3.1 (IOVDD), U3.10 (IOVDD), U3.22 (IOVDD), U3.33 (IOVDD), U3.42 (IOVDD), U3.43 (ADC_AVDD), U3.44 (VREG_IN), U3.48 (USB_VDD), U3.49 (IOVDD), C35.1, C36.1, C38.1, C39.1, C40.1
- removed net V_{MCU}: C11.1, C14.1, C17.1, C19.1, C20.1, U3.1 (IOVDD), U3.10 (IOVDD), U3.22 (IOVDD), U3.33 (IOVDD), U3.42 (IOVDD), U3.43 (ADC_AVDD), U3.44 (VREG_IN), U3.48 (USB_VDD), U3.49 (IOVDD)
- no-connect marks 1 -> 4
Other:
- moved on the sheet: C12, C14, C16, C17, C19, C20, R16, R17, R20, R21, R23, R24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

Commit message: ok for rp2040
Parts:
- added SW2: Reset, Button_Switch_SMD:SW_SPST_EVQP2, symbol Switch:SW_Push
Connections:
- net GND: now also SW2.2
- net RUN: now reaches U3.26 (RUN)
- net RUN: now also SW2.1
- no-connect marks 4 -> 2
Other:
- moved on the sheet: R22, R25
Changed lines of the file:
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@@
 		(at 175.26 147.32)
 	)
-	(no_connect
-		(at 27.94 97.79)
-	)
-	(no_connect
-		(at 86.36 172.72)
-	)
 	(bus_entry
 		(at 93.98 134.62)
@@
 	(wire
 		(pts
-			(xy 115.57 81.28) (xy 124.46 81.28)
+			(xy 113.03 81.28) (xy 124.46 81.28)
 		)
 		(stroke
@@
 	(wire
 		(pts
+			(xy 53.34 100.33) (xy 53.34 97.79)
+		)
+		(stroke
+			(width 0)
+			(type default)
+		)
+	)
+	(wire
+		(pts
 			(xy 175.26 99.06) (xy 198.12 99.06)
 		)
@@
 	(wire
 		(pts
+			(xy 118.11 71.12) (xy 124.46 71.12)
+		)
+		(stroke
+			(width 0)
+			(type default)
+		)
+	)
+	(wire
+		(pts
 			(xy 96.52 93.98) (xy 124.46 93.98)
 		)
@@
 	(wire
 		(pts
+			(xy 53.34 85.09) (xy 53.34 87.63)
+		)
+		(stroke
+			(width 0)
+			(type default)
+		)
+	)
+	(wire
+		(pts
 			(xy 229.87 38.1) (xy 240.03 38.1)
 		)
@@
 	(wire
 		(pts
-			(xy 119.38 73.66) (xy 115.57 73.66)
+			(xy 119.38 73.66) (xy 113.03 73.66)
 		)
 		(stroke
@@
 	(wire
 		(pts
-			(xy 96.52 73.66) (xy 107.95 73.66)
+			(xy 96.52 73.66) (xy 105.41 73.66)
 		)
 		(stroke
@@
 	(wire
 		(pts
-			(xy 96.52 81.28) (xy 107.95 81.28)
+			(xy 96.52 81.28) (xy 105.41 81.28)
 		)
 		(stroke
@@
 		)
 	)
+	(label "RUN"
+		(at 118.11 71.12 180)
+		(fields_autoplaced yes)
+		(effects
+			(font
+				(size 1.27 1.27)
+			)
+			(justify right bottom)
+		)
+	)
 	(label "FLASH.IO1"
 		(at 106.68 96.52 180)
@@
 		)
 	)
+	(label "RUN"
+		(at 53.34 85.09 90)
+		(fields_autoplaced yes)
+		(effects
+			(font
+				(size 1.27 1.27)
+			)
+			(justify left bottom)
+		)
+	)
 	(label "FLASH.IO2"
 		(at 106.68 99.06 180)
@@
 	(symbol
 		(lib_id "Device:R")
-		(at 111.76 81.28 270)
+		(at 109.22 81.28 270)
 		(unit 1)
 		(exclude_from_sim no)
@@
 		(dnp no)
 		(property "Reference" "R25"
-			(at 111.76 76.454 90)
+			(at 109.22 76.454 90)
 			(effects
 				(font
@@
 		)
 		(property "Value" "27.4"
-			(at 111.76 78.994 90)
+			(at 109.22 78.994 90)
 			(effects
 				(font
@@
 		)
 		(property "Footprint" "Resistor_SMD:R_0603_1608Metric"
-			(at 111.76 79.502 90)
+			(at 109.22 79.502 90)
 			(effects
 				(font
@@
 		)
 		(property "Datasheet" "~"
-			(at 111.76 81.28 0)
+			(at 109.22 81.28 0)
 			(effects
 				(font
@@
 		)
 		(property "Description" ""
-			(at 111.76 81.28 0)
+			(at 109.22 81.28 0)
 			(effects
 				(font
@@
 		)
 		(property "MPN" ""
-			(at 111.76 81.28 0)
+			(at 109.22 81.28 0)
 			(effects
 				(font
@@
 		)
 		(property "Manufacturer" ""
-			(at 111.76 81.28 0)
+			(at 109.22 81.28 0)
 			(effects
 				(font
@@
 	)
 	(symbol
+		(lib_id "Switch:SW_Push")
+		(at 53.34 92.71 270)
+		(unit 1)
+		(exclude_from_sim no)
+		(in_bom yes)
+		(on_board yes)
+		(dnp no)
+		(fields_autoplaced yes)
+		(property "Reference" "SW2"
+			(at 57.15 91.4399 90)
+			(effects
+				(font
+					(size 1.27 1.27)
+				)
+				(justify left)
+			)
+		)
+		(property "Value" "Reset"
+			(at 57.15 93.9799 90)
+			(effects
+				(font
+					(size 1.27 1.27)
+				)
+				(justify left)
+			)
+		)
+		(property "Footprint" "Button_Switch_SMD:SW_SPST_EVQP2"
+			(at 58.42 92.71 0)
+			(effects
+				(font
+					(size 1.27 1.27)
+				)
+				(hide yes)
+			)
+		)
+		(property "Datasheet" "~"
+			(at 58.42 92.71 0)
+			(effects
+				(font
+					(size 1.27 1.27)
+				)
+				(hide yes)
+			)
+		)
+		(property "Description" ""
+			(at 53.34 92.71 0)
+			(effects
+				(font
+					(size 1.27 1.27)
+				)
+				(hide yes)
+			)
+		)
+		(property "MPN" "EVQ-P2602W"
+			(at 53.34 92.71 0)
+			(effects
+				(font
+					(size 1.27 1.27)
+				)
+				(hide yes)
+			)
+		)
+		(property "Manufacturer" "Panasonic"
+			(at 53.34 92.71 0)
+			(effects
+				(font
+					(size 1.27 1.27)
+				)
+				(hide yes)
+			)
+		)
+		(pin "1"
+		)
+		(pin "2"
+		)
+		(instances
+			(project "Tattoo_Supply"
+				(path "/036b57f3-323c-4da7-bad2-1c27fa1415e1/fd65dc63-1d27-4821-ae4f-326fe3a44815"
+					(reference "SW2")
+					(unit 1)
+				)
+			)
+		)
+	)
+	(symbol
 		(lib_id "power:GND")
 		(at 133.35 54.61 0)
@@
 	(symbol
 		(lib_id "Device:R")
-		(at 111.76 73.66 270)
+		(at 109.22 73.66 270)
 		(unit 1)
 		(exclude_from_sim no)
@@
 		(dnp no)
 		(property "Reference" "R22"
-			(at 112.014 68.834 90)
+			(at 109.474 68.834 90)
 			(effects
 				(font
@@
 		)
 		(property "Value" "27.4"
-			(at 112.014 71.374 90)
+			(at 109.474 71.374 90)
 			(effects
 				(font
@@
 		)
 		(property "Footprint" "Resistor_SMD:R_0603_1608Metric"
-			(at 111.76 71.882 90)
+			(at 109.22 71.882 90)
 			(effects
 				(font
@@
 		)
 		(property "Datasheet" "~"
-			(at 111.76 73.66 0)
+			(at 109.22 73.66 0)
 			(effects
 				(font
@@
 		)
 		(property "Description" ""
-			(at 111.76 73.66 0)
+			(at 109.22 73.66 0)
 			(effects
 				(font
@@
 		)
 		(property "MPN" ""
-			(at 111.76 73.66 0)
+			(at 109.22 73.66 0)
 			(effects
 				(font
@@
 		)
 		(property "Manufacturer" ""
-			(at 111.76 73.66 0)
+			(at 109.22 73.66 0)
 			(effects
 				(font
@@
 					(unit 1)
 				)
+			)
+		)
+	)
+	(symbol
+		(lib_id "power:GND")
+		(at 53.34 100.33 0)
+		(unit 1)
+		(exclude_from_sim no)
+		(in_bom yes)
+		(on_board yes)
+		(dnp no)
+		(fields_autoplaced yes)
+		(property "Reference" "#PWR076"
+			(at 53.34 106.68 0)
+			(effects
+				(font
+					(size 1.27 1.27)
+				)
+				(hide yes)
+			)
+		)
+		(property "Value" "GND"
+			(at 53.34 105.41 0)
+			(effects
+				(font
+					(size 1.27 1.27)
+				)
+			)
+		)
+		(property "Footprint" ""
+			(at 53.34 100.33 0)
+			(effects
+				(font
+					(size 1.27 1.27)
+				)
+				(hide yes)
+			)
+		)
+		(property "Datasheet" ""
+			(at 53.34 100.33 0)
+			(effects
+				(font
+					(size 1.27 1.27)
+				)
+				(hide yes)
+			)
+		)
+		(property "Description" ""
+			(at 53.34 100.33 0)
+			(effects
+				(font
+					(size 1.27 1.27)
+				)
+				(hide yes)
+			)
+		)
+		(pin "1"
+		)
+		(instances
+			(project "Tattoo_Supply"
+				(path "/036b57f3-323c-4da7-bad2-1c27fa1415e1/fd65dc63-1d27-4821-ae4f-326fe3a44815"
+					(reference "#PWR076")
+					(unit 1)
+				)

Commit message: ok for dcdc and cleanup
Parts:
- R21: value 10k -> 100k; MPN ERJ-3EKF1002V -> (none); Manufacturer Panasonic -> (none)
Connections:
- net 3V3: no longer R21.1
- net GND: now also R21.1
Changed lines of the file:
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@@
+	(wire
+		(pts
+			(xy 208.28 102.87) (xy 208.28 104.14)
+		)
+		(stroke
+			(width 0)
+			(type default)
+		)
+	)
 	(wire
 		(pts
@@
 		(shape output)
 		(at 208.28 99.06 0)
-		(fields_autoplaced yes)
-		(effects
-			(font
-				(size 1.27 1.27)
-			)
-			(justify left)
-		)
-	)
-	(hierarchical_label "3V3"
-		(shape input)
-		(at 208.28 102.87 0)
 		(fields_autoplaced yes)
 		(effects
@@
 				(path "/036b57f3-323c-4da7-bad2-1c27fa1415e1/fd65dc63-1d27-4821-ae4f-326fe3a44815"
 					(reference "Y1")
+					(unit 1)
+				)
+			)
+		)
+	)
+	(symbol
+		(lib_id "power:GND")
+		(at 208.28 104.14 0)
+		(unit 1)
+		(exclude_from_sim no)
+		(in_bom yes)
+		(on_board yes)
+		(dnp no)
+		(fields_autoplaced yes)
+		(property "Reference" "#PWR026"
+			(at 208.28 110.49 0)
+			(effects
+				(font
+					(size 1.27 1.27)
+				)
+				(hide yes)
+			)
+		)
+		(property "Value" "GND"
+			(at 208.28 109.22 0)
+			(effects
+				(font
+					(size 1.27 1.27)
+				)
+			)
+		)
+		(property "Footprint" ""
+			(at 208.28 104.14 0)
+			(effects
+				(font
+					(size 1.27 1.27)
+				)
+				(hide yes)
+			)
+		)
+		(property "Datasheet" ""
+			(at 208.28 104.14 0)
+			(effects
+				(font
+					(size 1.27 1.27)
+				)
+				(hide yes)
+			)
+		)
+		(property "Description" ""
+			(at 208.28 104.14 0)
+			(effects
+				(font
+					(size 1.27 1.27)
+				)
+				(hide yes)
+			)
+		)
+		(pin "1"
+		)
+		(instances
+			(project "Tattoo_Supply"
+				(path "/036b57f3-323c-4da7-bad2-1c27fa1415e1/fd65dc63-1d27-4821-ae4f-326fe3a44815"
+					(reference "#PWR026")
 					(unit 1)
 				)
@@
 			)
 		)
-		(property "Value" "10k"
+		(property "Value" "100k"
 			(at 203.2 107.696 90)
 			(effects
@@
 			)
 		)
-		(property "MPN" "ERJ-3EKF1002V"
+		(property "MPN" ""
 			(at 203.2 102.87 0)
 			(effects
@@
 			)
 		)
-		(property "Manufacturer" "Panasonic"
+		(property "Manufacturer" ""
 			(at 203.2 102.87 0)
 			(effects

Commit message: ok for efuse w/o values
Parts:
- removed R23, R24: 20, Resistor_SMD:R_0603_1608Metric, symbol Device:R
Connections:
- net SW1: now also U3.11 (GPIO8)
- net SW2: now also U3.12 (GPIO9)
Changed lines of the file:
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@@
 	(wire
 		(pts
-			(xy 175.26 93.98) (xy 190.5 93.98)
+			(xy 175.26 93.98) (xy 181.61 93.98)
 		)
 		(stroke
@@
 	(wire
 		(pts
-			(xy 198.12 91.44) (xy 208.28 91.44)
-		)
-		(stroke
-			(width 0)
-			(type default)
-		)
-	)
-	(wire
-		(pts
 			(xy 240.03 38.1) (xy 240.03 40.64)
 		)
@@
 	(wire
 		(pts
-			(xy 198.12 93.98) (xy 208.28 93.98)
-		)
-		(stroke
-			(width 0)
-			(type default)
-		)
-	)
-	(wire
-		(pts
 			(xy 175.26 71.12) (xy 203.2 71.12)
 		)
@@
 	(wire
 		(pts
-			(xy 175.26 91.44) (xy 190.5 91.44)
+			(xy 175.26 91.44) (xy 181.61 91.44)
 		)
 		(stroke
@@
 	(hierarchical_label "SW1"
 		(shape output)
-		(at 208.28 91.44 0)
+		(at 181.61 91.44 0)
 		(fields_autoplaced yes)
 		(effects
@@
 	(hierarchical_label "SW2"
 		(shape output)
-		(at 208.28 93.98 0)
+		(at 181.61 93.98 0)
 		(fields_autoplaced yes)
 		(effects
@@
 	)
 	(symbol
-		(lib_id "Device:R")
-		(at 194.31 93.98 90)
-		(unit 1)
-		(exclude_from_sim no)
-		(in_bom yes)
-		(on_board yes)
-		(dnp no)
-		(property "Reference" "R24"
-			(at 199.136 92.71 90)
-			(effects
-				(font
-					(size 1.27 1.27)
-				)
-			)
-		)
-		(property "Value" "20"
-			(at 194.31 93.98 90)
-			(effects
-				(font
-					(size 1.27 1.27)
-				)
-			)
-		)
-		(property "Footprint" "Resistor_SMD:R_0603_1608Metric"
-			(at 194.31 95.758 90)
-			(effects
-				(font
-					(size 1.27 1.27)
-				)
-				(hide yes)
-			)
-		)
-		(property "Datasheet" "~"
-			(at 194.31 93.98 0)
-			(effects
-				(font
-					(size 1.27 1.27)
-				)
-				(hide yes)
-			)
-		)
-		(property "Description" ""
-			(at 194.31 93.98 0)
-			(effects
-				(font
-					(size 1.27 1.27)
-				)
-				(hide yes)
-			)
-		)
-		(property "MPN" "ERJ-3EKF20R0V"
-			(at 194.31 93.98 0)
-			(effects
-				(font
-					(size 1.27 1.27)
-				)
-				(hide yes)
-			)
-		)
-		(property "Manufacturer" "Panasonic"
-			(at 194.31 93.98 0)
-			(effects
-				(font
-					(size 1.27 1.27)
-				)
-				(hide yes)
-			)
-		)
-		(pin "1"
-		)
-		(pin "2"
-		)
-		(instances
-			(project "Tattoo_Supply"
-				(path "/036b57f3-323c-4da7-bad2-1c27fa1415e1/fd65dc63-1d27-4821-ae4f-326fe3a44815"
-					(reference "R24")
-					(unit 1)
-				)
-			)
-		)
-	)
-	(symbol
 		(lib_id "power:GND")
 		(at 53.34 100.33 0)
@@
 					(unit 1)
 				)
-			)
-		)
-	)
-	(symbol
-		(lib_id "Device:R")
-		(at 194.31 91.44 90)
-		(unit 1)
-		(exclude_from_sim no)
-		(in_bom yes)
-		(on_board yes)
-		(dnp no)
-		(property "Reference" "R23"
-			(at 199.136 90.17 90)
-			(effects
-				(font
-					(size 1.27 1.27)
-				)
-			)
-		)
-		(property "Value" "20"
-			(at 194.31 91.44 90)
-			(effects
-				(font
-					(size 1.27 1.27)
-				)
-			)
-		)
-		(property "Footprint" "Resistor_SMD:R_0603_1608Metric"
-			(at 194.31 93.218 90)
-			(effects
-				(font
-					(size 1.27 1.27)
-				)
-				(hide yes)
-			)
-		)
-		(property "Datasheet" "~"
-			(at 194.31 91.44 0)
-			(effects
-				(font
-					(size 1.27 1.27)
-				)
-				(hide yes)
-			)
-		)
-		(property "Description" ""
-			(at 194.31 91.44 0)
-			(effects
-				(font
-					(size 1.27 1.27)
-				)
-				(hide yes)
-			)
-		)
-		(property "MPN" "ERJ-3EKF20R0V"
-			(at 194.31 91.44 0)
-			(effects
-				(font
-					(size 1.27 1.27)
-				)
-				(hide yes)
-			)
-		)
-		(property "Manufacturer" "Panasonic"
-			(at 194.31 91.44 0)
-			(effects
-				(font
-					(size 1.27 1.27)
-				)
-				(hide yes)
-			)
-		)
-		(pin "1"
-		)
-		(pin "2"
-		)
-		(instances
-			(project "Tattoo_Supply"
-				(path "/036b57f3-323c-4da7-bad2-1c27fa1415e1/fd65dc63-1d27-4821-ae4f-326fe3a44815"
-					(reference "R23")
-					(unit 1)
-				)
